File: pcb/befour.kicad_sch (KiCad schematic)
At the start: 8 parts, among them SW1 SW_SPDT, U1 74LS374, U2 MEMORY, U3 74LS161, U4 74LS138, U5 AREG, X1 1MHz

Commit message: more pcb work
Parts:
- removed R8: 1k, symbol Device:R
- removed SW1: SW_SPDT, symbol Switch:SW_SPDT
- added D1, D2: D, Diode_THT:D_DO-35_SOD27_P7.62mm_Horizontal, symbol Device:D
- added R1: 10k, Resistor_THT:R_Axial_DIN0207_L6.3mm_D2.5mm_P10.16mm_Horizontal, symbol Device:R
- added SW1: SW_Push, Button_Switch_THT:SW_PUSH_6mm_H5mm, symbol Switch:SW_Push
- added SW2: SW_SPDT, Button_Switch_THT:SW_Slide_SPDT_Straight_CK_OS102011MS2Q, symbol Switch:SW_SPDT
- added U11: TEMP, Package_DIP:DIP-16_W7.62mm_Socket, symbol 74xx:74LS161
- added U12: BREG, Package_DIP:DIP-16_W7.62mm_Socket, symbol 74xx:74LS161
- added U2, U3: 74LS125, Package_DIP:DIP-14_W7.62mm_Socket, symbol 74xx:74LS125
- added U5: 74LS14, Package_DIP:DIP-14_W7.62mm_Socket, symbol 74xx:74LS14
- added U6: 74LS138, Package_DIP:DIP-16_W7.62mm_Socket, symbol 74xx:74LS138
- added U8: 74LS11, Package_DIP:DIP-14_W7.62mm_Socket, symbol 74xx:74LS11
- U10: renamed from U5; footprint (none) -> Package_DIP:DIP-16_W7.62mm_Socket
- U4: renamed from U1; footprint (none) -> Package_DIP:DIP-20_W7.62mm_Socket
- U7: renamed from U3; footprint (none) -> Package_DIP:DIP-16_W7.62mm_Socket
- U9: renamed from U4; footprint (none) -> Package_DIP:DIP-16_W7.62mm_Socket
- renumbered U2 to U1
Connections:
- net +5V: now also R1.2, U11.16 (VCC), U12.16 (VCC), U2.14 (VCC), U3.14 (VCC), U5.14 (VCC), U6.16 (VCC), U6.6 (E3), U8.14 (VCC), U8.2, U8.4
- net DATABUS0: now also U11.3 (D0), U12.3 (D0), U3.2
- net DATABUS1: now also U11.4 (D1), U12.4 (D1), U3.5
- net DATABUS2: now also U11.5 (D2), U12.5 (D2), U3.9
- net DATABUS3: now also U11.6 (D3), U12.6 (D3), U3.12
- net GND: now also U10.10 (CET), U10.7 (CEP), U4.1 (OE), X1.1 (EN), SW1.1, U11.10 (CET), U11.7 (CEP), U11.8 (GND), U12.10 (CET), U12.7 (CEP), U12.8 (GND), U2.7 (GND), U3.7 (GND), U5.7 (GND), U6.5 (E2), U6.8 (GND), U8.7 (GND)
- net LDINST: now also U5.11
- net RESET: now also U10.1 (~{MR}), U11.1 (~{MR}), U12.1 (~{MR}), U6.4 (E1)
- net ROM0: now also U2.3; no longer U1.11 (Q0), U4.3 (D0)
- net ROM1: now also U2.6; no longer U1.12 (Q1), U4.4 (D1)
- net ROM2: now also U2.8; no longer U1.13 (Q2), U4.7 (D2)
- net ROM3: now also U2.11; no longer U1.15 (Q3), U4.8 (D3)
- net ROM4: now also U3.3; no longer U1.16 (Q4), U4.13 (D4)
- net ROM5: now also U3.6; no longer U1.17 (Q5), U4.14 (D5)
- net ROM6: now also U3.8; no longer U1.18 (Q6), U4.17 (D6)
- net ROM7: now also U3.11; no longer U1.19 (Q7), U4.18 (D7)
- net nLDINST: now reaches U4.11 (Cp)
- net nLDINST: now also U5.10
- net SI0: now reaches U4.12 (O4)
- net SI1: now reaches U4.15 (O5)
- net SI2: now reaches U4.16 (O6)
- net SI3: now reaches U4.19 (O7)
- net at U4.2 (O0): now also U6.1 (A0)
- net at U4.5 (O1): now also U6.2 (A1)
- net at U4.6 (O2): now also U6.3 (A2)
- net AB: now reaches U4.9 (O3)
- net ROMnCS: now reaches U1.20 (~{CS})
- net at U1.22 (~{OE}): now also U5.2
- net WRITE: now reaches U1.27 (~{WE})
- net WRITE: now also D1.1 (K), D2.1 (K), U2.1, U2.10, U2.13, U2.4, U3.1, U3.10, U3.13, U3.4, U5.1
- net CLK: now reaches U10.2 (CP)
- net CLK: now also X1.8 (OUT), SW2.3 (C), U12.2 (CP)
- net writeA: now reaches U10.9 (~{PE})
- net at U7.2 (CP): now also SW2.2 (B); no longer X1.8 (OUT)
- new net: R1.1, SW1.2, SW2.1 (A)
- new net ADD: U6.13 (O2), U8.13
- new net ADDRESSING: U8.6
- new net ALUOP: U11.9 (~{PE}), U8.12
- new net BOUT0: U12.14 (Q0), U2.2
- new net BOUT1: U12.13 (Q1), U2.5
- new net BOUT2: U12.12 (Q2), U2.9
- new net BOUT3: U12.11 (Q3), U2.12
- new net CMP: U6.11 (O4)
- new net D0: U1.11 (Q0), U4.3 (D0)
- new net D1: U1.12 (Q1), U4.4 (D1)
- new net D2: U1.13 (Q2), U4.7 (D2)
- new net D3: U1.15 (Q3), U4.8 (D3)
- new net D4: U1.16 (Q4), U4.13 (D4)
- new net D5: U1.17 (Q5), U4.14 (D5)
- new net D6: U1.18 (Q6), U4.17 (D6)
- new net D7: U1.19 (Q7), U4.18 (D7)
- new net JP: U6.9 (O6)
- new net JPC: U6.7 (O7)
- new net LD: U6.14 (O1), U8.3
- new net LDI: U6.15 (O0)
- new net NAND: U6.12 (O3), U8.1
- new net OP1^: U11.2 (CP)
- new net OPERATION: D2.2 (A)
- new net ST: D1.2 (A), U6.10 (O5), U8.5
- new net TEMPOUT0: U11.14 (Q0)
- new net TEMPOUT1: U11.13 (Q1)
- new net TEMPOUT2: U11.12 (Q2)
- new net TEMPOUT3: U11.11 (Q3)
- new net writeB: U12.9 (~{PE})

Commit message: the Schematic is complete.
Parts:
- added D10, D11, D12, D13, D14, D15, D16, D17, D18, D19, D20, D21, D22, D23, D24, D25, D26, D27, D28, D29, D3, D30, D31, D32, D33, D34, D35, D36, D37, D38, D39, D4, D40, D41, D42, D43, D44, D45, D46, D47, D48, D49, D5, D50, D51, D52, D53, D54, D55, D6, D7, D8, D9: D, Diode_THT:D_DO-35_SOD27_P2.54mm_Vertical_KathodeUp, symbol Device:D
- added J1: USB_C_Receptacle_PowerOnly_6P, Connector_USB:USB_C_Receptacle_GCT_USB4125-xx-x_6P_TopMnt_Horizontal, symbol Connector:USB_C_Receptacle_PowerOnly_6P
- added J2: READOUT, Connector_PinHeader_2.54mm:PinHeader_1x16_P2.54mm_Vertical, symbol Connector:Conn_01x16_Pin
- added J3: DEVICES, Connector_PinHeader_2.54mm:PinHeader_1x05_P2.54mm_Vertical, symbol Connector:Conn_01x05_Pin
- added R1: 1k, Resistor_THT:R_Axial_DIN0207_L6.3mm_D2.5mm_P10.16mm_Horizontal, symbol Device:R
- added R10, R4, R5, R6, R7, R8, R9: 10K, Resistor_THT:R_Axial_DIN0207_L6.3mm_D2.5mm_P10.16mm_Horizontal, symbol Device:R
- added R11: 10k, Resistor_THT:R_Axial_DIN0207_L6.3mm_D2.5mm_P10.16mm_Horizontal, symbol Device:R
- added R2, R3: 5.1K, Resistor_THT:R_Axial_DIN0207_L6.3mm_D2.5mm_P10.16mm_Horizontal, symbol Device:R
- added SW1: SW_SPDT, Connector_PinHeader_2.54mm:PinHeader_1x03_P2.54mm_Vertical, symbol Switch:SW_SPDT
- added SW2: PRG_SELECT, Button_Switch_SMD:SW_DIP_SPSTx08_Slide_9.78x22.5mm_W8.61mm_P2.54mm, symbol Switch:SW_DIP_x08
- added SW3: SW_Push, Button_Switch_THT:SW_PUSH_6mm_H5mm, symbol Switch:SW_Push
- added U10, U20: 74LS11, Package_DIP:DIP-14_W7.62mm_Socket, symbol 74xx:74LS11
- added U11: ALU_ADD, Package_DIP:DIP-16_W7.62mm_Socket, symbol 74xx:74LS283
- added U12: ALU_NAND, Package_DIP:DIP-14_W7.62mm_Socket, symbol 74xx:74LS00
- added U13: SI_BUFFER, Package_DIP:DIP-14_W7.62mm_Socket, symbol 74xx:74LS125
- added U14, U25: 74LS00, Package_DIP:DIP-14_W7.62mm_Socket, symbol 74xx:74LS00
- added U16: 74LS14, Package_DIP:DIP-14_W7.62mm_Socket, symbol 74xx:74LS14
- added U17: MISC, Package_DIP:DIP-14_W7.62mm_Socket, symbol 74xx:74LS125
- added U18: ALU_NAND_BUFFER, Package_DIP:DIP-14_W7.62mm_Socket, symbol 74xx:74LS125
- added U21: A_BUFFER, Package_DIP:DIP-14_W7.62mm_Socket, symbol 74xx:74LS125
- added U22: ALU_ADD_BUFFER, Package_DIP:DIP-14_W7.62mm_Socket, symbol 74xx:74LS125
- added U26: XOR_EQUAL, Package_DIP:DIP-14_W7.62mm_Socket, symbol 74xx:74LS136
- added U29: FLAGS_BUFFER, Package_DIP:DIP-14_W7.62mm_Socket, symbol 74xx:74LS125
- added U30: DEVICES_BUFFER, Package_DIP:DIP-14_W7.62mm_Socket, symbol 74xx:74LS125
- added U31: PCH_BUFFER, Package_DIP:DIP-14_W7.62mm_Socket, symbol 74xx:74LS125
- added U32: 74LS138, Package_DIP:DIP-16_W7.62mm_Socket, symbol 74xx:74LS138
- added U33: PCL_BUFFER, Package_DIP:DIP-14_W7.62mm_Socket, symbol 74xx:74LS125
- added U34: PCH, Package_DIP:DIP-16_W7.62mm_Socket, symbol 74xx:74LS161
- added U35: PCL, Package_DIP:DIP-16_W7.62mm_Socket, symbol 74xx:74LS161
- added U36: ADR_BUFFER, Package_DIP:DIP-14_W7.62mm_Socket, symbol 74xx:74LS125
- added U37: SI_ADR_BUFFER, Package_DIP:DIP-14_W7.62mm_Socket, symbol 74xx:74LS125
- added U6: TEMP_BUFFER, Package_DIP:DIP-14_W7.62mm_Socket, symbol 74xx:74LS125
- added U7: B_BUFFER, Package_DIP:DIP-14_W7.62mm_Socket, symbol 74xx:74LS125
- added U8: 74LS125, Package_DIP:DIP-14_W7.62mm_Socket, symbol 74xx:74LS125
- D1, D2: footprint Diode_THT:D_DO-35_SOD27_P7.62mm_Horizontal -> Diode_THT:D_DO-35_SOD27_P2.54mm_Vertical_KathodeUp
- U15: renamed from U7; value 74LS161 -> CLKDIV
- U23: renamed from U9; value 74LS138 -> CLKDIV2
- U3: renamed from U2; value 74LS125 -> B_OUT_BUFFER
- U4: renamed from U3; value 74LS125 -> DB_OUT_BUFFER
- U5: renamed from U4; value 74LS374 -> INSTSTORe
- renumbered R1 to R12, SW1 to SW4, SW2 to SW5, U5 to U1, U8 to U19, U1 to U2, U10 to U24, U11 to U27, U12 to U28, U6 to U9
Connections:
- net OP1^ is gone; now on net OP1: U27.2 (CP)
- net ROM0 is gone; now on net D0: U3.3
- net ROM1 is gone; now on net D1: U3.6
- net ROM2 is gone; now on net D2: U3.8
- net ROM3 is gone; now on net D3: U3.11
- net ROM4 is gone; now on net D4: U4.3
- net ROM5 is gone; now on net D5: U4.6
- net ROM6 is gone; now on net D6: U4.8
- net ROM7 is gone; now on net D7: U4.11
- net +5V: now also R11.2, SW1.2 (B), SW2.1, SW2.2, SW2.3, SW2.4, SW2.5, SW2.6, SW2.7, SW2.8, U10.14 (VCC), U10.4, U11.16 (VCC), U12.14 (VCC), U13.14 (VCC), U14.14 (VCC), U16.14 (VCC), U17.14 (VCC), U18.14 (VCC), U20.14 (VCC), U20.2, U21.14 (VCC), U22.14 (VCC), U25.14 (VCC), U26.14 (VCC), U29.14 (VCC), U29.2, U30.14 (VCC), U31.14 (VCC), U32.16 (VCC), U32.6 (E3), U33.14 (VCC), U34.10 (CET), U34.16 (VCC), U35.10 (CET), U35.16 (VCC), U36.12, U36.14 (VCC), U36.2, U36.5, U36.9, U37.14 (VCC), U6.14 (VCC), U7.14 (VCC), U8.14 (VCC); no longer U19.2, U19.4
- net AB: now also U1.3, U19.10, U19.9, D4.2 (A), D43.2 (A)
- net ADD: now also U14.9, U16.3, U18.1, U22.1, U22.10, U22.13, U22.4
- net ADDRESSING: now also D16.2 (A)
- net ALUOP: now also D14.2 (A), D9.2 (A)
- net AOUT0: now also D33.2 (A), J2.1 (Pin_1), U11.5 (A1), U12.1, U21.12, U26.13
- net AOUT1: now also D32.2 (A), J2.2 (Pin_2), U11.3 (A2), U12.4, U21.9, U26.10
- net AOUT2: now also D31.2 (A), J2.3 (Pin_3), U11.14 (A3), U12.9, U21.5, U26.5
- net BOUT0: now also J2.5 (Pin_5), U26.12, U6.12
- net BOUT1: now also J2.6 (Pin_6), U26.9, U6.9
- net BOUT2: now also J2.7 (Pin_7), U26.4, U7.5
- net BOUT3: now also J2.8 (Pin_8), U26.1, U7.2
- net CMP: now also U14.10, U17.4, U32.5 (E2)
- net D4: now also U8.12
- net D5: now also U8.9
- net D6: now also U8.5
- net D7: now also U8.2
- net GND: now also J1.A12 (GND), J1.B12 (GND), J1.S1 (SHIELD), R1.2, R10.2, R2.1, R3.1, R4.2, R5.2, R6.2, R7.2, R8.2, R9.2, SW3.1, U10.7 (GND), U11.8 (GND), U12.7 (GND), U13.7 (GND), U14.7 (GND), U16.7 (GND), U17.7 (GND), U18.7 (GND), U20.7 (GND), U21.7 (GND), U22.7 (GND), U25.7 (GND), U26.7 (GND), U29.7 (GND), U30.7 (GND), U31.7 (GND), U32.4 (E1), U32.8 (GND), U33.7 (GND), U34.8 (GND), U35.8 (GND), U36.7 (GND), U37.7 (GND), U6.7 (GND), U7.7 (GND), U8.7 (GND); no longer U2.1 (A14), U2.2 (A12), U2.21 (A10), U2.23 (A11), U2.24 (A9), U2.25 (A8), U2.26 (A13)
- net INCPC: now also U14.4
- net JP: now also U20.10, U20.9
- net JPC: now also D28.2 (A)
- net LD: now also U19.4, D12.2 (A), U10.1, U10.2
- net LDI: now also U10.13
- net NAND: now also U19.2
- net OP1: now also D11.2 (A), D19.2 (A), U10.3
- net OP2: now also D15.2 (A), D24.2 (A), D27.2 (A), D39.2 (A), D40.2 (A), U10.5, U14.5
- net OPERATION: now also D13.2 (A), D17.2 (A), D5.2 (A), D8.2 (A), U10.6
- net RESET: now also R11.1, SW3.2, U20.4, U20.5, U34.1 (~{MR})
- net ROMnCS: now also J3.5 (Pin_5)
- net SI0: now also U13.12, U32.1 (A0), U34.6 (D3), U35.6 (D3), U37.12
- net SI1: now also U13.9, U32.2 (A1), U34.5 (D2), U35.5 (D2), U37.9
- net SI2: now also U13.5, U32.3 (A2), U34.4 (D1), U35.4 (D1), U37.5
- net SI3: now also U13.2, U34.3 (D0), U35.3 (D0), U37.2
- net ST: now also D3.2 (A), D6.2 (A)
- net TEMPOUT0: now also U7.12
- net TEMPOUT1: now also U7.9
- net TEMPOUT2: now also U6.5
- net TEMPOUT3: now also U6.2
- net writeA: now also D25.1 (K), D26.1 (K), D27.1 (K)
- net writeB: now also D22.1 (K), D23.1 (K), D24.1 (K)
- net Inst0: now reaches U5.2 (O0), U9.1 (A0)
- net Inst1: now reaches U5.5 (O1), U9.2 (A1)
- net Inst1: now also U1.9
- net Inst2: now reaches U5.6 (O2), U9.3 (A2)
- net Inst2: now also D25.2 (A)
- net A0: now reaches U2.10 (A0)
- net A0: now also J2.9 (Pin_9), U33.11, U37.11
- net A7: now reaches U2.3 (A7)
- net A7: now also J2.16 (Pin_16), U31.3, U36.3
- net A6: now reaches U2.4 (A6)
- net A6: now also J2.15 (Pin_15), U31.6, U36.6
- net A5: now reaches U2.5 (A5)
- net A5: now also J2.14 (Pin_14), U31.8, U36.8
- net A4: now reaches U2.6 (A4)
- net A4: now also J2.13 (Pin_13), U31.11, U36.11
- net A3: now reaches U2.7 (A3)
- net A3: now also J2.12 (Pin_12), U33.3, U37.3
- net A2: now reaches U2.8 (A2)
- net A2: now also J2.11 (Pin_11), U33.6, U37.6
- net A1: now reaches U2.9 (A1)
- net A1: now also J2.10 (Pin_10), U33.8, U37.8
- net at U19.11: now also U1.8
- net at U19.8: now also D26.2 (A)
- net nAB: now reaches U1.4
- net nAB: now also D10.2 (A), D23.2 (A), D45.2 (A), D7.2 (A), U14.12, U14.13, U17.13
- net at U1.12: now also U34.7 (CEP)
- net PerformJump: now reaches U1.13
- net PerformJump: now also D38.1 (K), D39.1 (K), D41.2 (A), D42.2 (A), D44.2 (A), U35.7 (CEP)
- net at U1.5: now also D40.1 (K), D41.1 (K)
- net at U1.6: now also D46.2 (A)
- net AOUT3 renamed SignFlag
- net SignFlag: now also D30.2 (A), J2.4 (Pin_4), U11.12 (A4), U12.12, U21.2, U26.2, U29.12
- net DATABUS0 renamed DB0
- net DB0: now also U11.6 (B1), U12.2, U13.11, U21.11, U6.11, U7.11, U8.11; no longer U27.3 (D0)
- net DATABUS1 renamed DB1
- net DB1: now also U11.2 (B2), U12.5, U13.8, U21.8, U6.8, U7.8, U8.8; no longer U27.4 (D1)
- net DATABUS2 renamed DB2
- net DB2: now also U11.15 (B3), U12.10, U13.6, U21.6, U6.6, U7.6, U8.6; no longer U27.5 (D2)
- net DATABUS3 renamed DB3
- net DB3: now also U11.11 (B4), U12.13, U13.3, U21.3, U6.3, U7.3, U8.3; no longer U27.6 (D3)
- new net: D48.1 (K), D49.1 (K), D50.1 (K), D51.1 (K), D52.1 (K), D53.1 (K), D54.1 (K), D55.1 (K), U17.12, U17.9
- new net: D48.2 (A), U30.11
- new net: D18.2 (A), U16.10
- new net: U14.8, U16.11
- new net: U30.4, U32.10 (O5)
- new net: D50.2 (A), U30.6
- new net: D6.1 (K), D7.1 (K), D8.1 (K), U20.1
- new net: D46.1 (K), D47.1 (K), U34.2 (CP)
- new net: U12.11, U18.12
- new net: D10.1 (K), D11.1 (K), D9.1 (K), U20.13
- new net: D20.1 (K), D21.1 (K), U16.5, U25.1
- new net: D18.1 (K), D19.1 (K), U25.2, U25.4
- new net: U25.3, U25.9
- new net: D42.1 (K), D43.1 (K), U35.9 (~{PE})
- new net: U11.13 (S3), U22.9
- new net: U11.10 (S4), U22.12
- new net: U14.6, U35.2 (CP)
- new net: U14.11, U17.10
- new net: U16.2, U31.1, U31.10, U31.13, U31.4, U33.1, U33.10, U33.13, U33.4
- new net: U31.9, U34.12 (Q2)
- new net: U33.2, U35.14 (Q0)
- new net: D30.1 (K), D31.1 (K), D32.1 (K), D33.1 (K), U16.9
- new net: D28.1 (K), D29.1 (K), U20.11
- new net: D22.2 (A), U10.12
- new net: R1.1, SW1.3 (C)
- new net: U16.6, U25.5
- new net: R10.1, SW2.10, U2.1 (A14)
- new net: R8.1, SW2.12, U2.2 (A12)
- new net: R6.1, SW2.14, U2.21 (A10)
- new net: R7.1, SW2.13, U2.23 (A11)
- new net: R5.1, SW2.15, U2.24 (A9)
- new net: R4.1, SW2.16, U2.25 (A8)
- new net: R9.1, SW2.11, U2.26 (A13)
- new net: U12.8, U18.9
- new net: D37.2 (A), U26.11
- new net: U11.1 (S2), U22.5
- new net: U11.4 (S1), U22.2
- new net: D34.1 (K), D35.1 (K), D36.1 (K), D37.1 (K), U16.13
- new net: D36.2 (A), U26.8
- new net: U25.13, U25.6
- new net: U31.12, U34.11 (Q3)
- new net: D53.2 (A), U29.8
- new net: D55.2 (A), U29.3
- new net: U30.10, U32.9 (O6)
- new net: D49.2 (A), U30.8
- new net: D20.2 (A), U18.3
- new net: U33.5, U35.13 (Q1)
- new net: U29.1, U32.15 (O0)
- new net: U16.4, U17.1, U18.10, U18.13, U18.4
- new net: J1.A9 (VBUS), J1.B9 (VBUS), SW1.1 (A)
- new net: D44.1 (K), D45.1 (K), U20.3, U34.9 (~{PE})
- new net: U20.6, U35.1 (~{MR})
- new net: D21.2 (A), U17.6
- new net: U12.6, U18.5
- new net: U33.12, U35.11 (Q3)
- new net: D47.2 (A), U35.15 (TC)
- new net: D34.2 (A), U26.3
- new net: U31.5, U34.13 (Q1)
- new net: U12.3, U17.2
- new net: U33.9, U35.12 (Q2)
- new net: D38.2 (A), U20.8
- new net: U31.2, U34.14 (Q0)
- new net: J1.A5 (CC1), R3.2
- new net: J1.B5 (CC2), R2.2
- new net: D54.2 (A), U29.6
- new net: U30.13, U32.7 (O7)
- new net: U29.4, U32.14 (O1)
- new net: U30.1, U32.11 (O4)
- new net: D51.2 (A), U30.3
- new net: U29.10, U32.13 (O2)
- new net: U10.8, U14.1
- new net: D35.2 (A), U26.6
- new net: U29.13, U32.12 (O3)
- new net: D52.2 (A), U29.11
- new net ALU0: U17.3, U22.3, U27.3 (D0)
- new net ALU1: U18.6, U22.6, U27.4 (D1)
- new net ALU2: U18.8, U22.8, U27.5 (D2)
- new net ALU3: U18.11, U22.11, U27.6 (D3)
- new net CIN: U11.7 (C0), U25.12, U25.8
- new net COUT: U11.9 (C4), U18.2
- new net CRES: U17.11, U17.5, U17.8
- new net Device0: J3.1 (Pin_1), U30.2
- new net Device1: J3.2 (Pin_2), U30.5
- new net Device2: J3.3 (Pin_3), U30.9
- new net Device3: J3.4 (Pin_4), U30.12
- new net EqualFlag: U16.12, U29.9
- new net MEMACCESS: D16.1 (K), D17.1 (K), U16.1, U36.1, U36.10, U36.13, U36.4, U37.1, U37.10, U37.13, U37.4
- new net ZeroFlag: U16.8, U29.5
- new net nCIN: D29.2 (A), U25.10, U25.11
- new net outputA: D3.1 (K), D4.1 (K), D5.1 (K), U10.11, U21.1, U21.10, U21.13, U21.4
- new net outputB: U10.10, U20.12, U6.10, U6.13, U7.1, U7.4
- new net outputLI: D12.1 (K), D13.1 (K), U10.9, U8.1, U8.10, U8.13, U8.4
- new net outputSI: U13.1, U13.10, U13.13, U13.4, U14.3
- new net outputTEMP: D14.1 (K), D15.1 (K), U14.2, U6.1, U6.4, U7.10, U7.13
- no-connect marks 0 -> 12
Other:
- moved on the sheet: U19C, U19D, U1B, U1C, U1D, U1E, U1F, U1G, U3E, U4E

Commit message: Update befour.kicad_sch
Other:
- note added: "TODO: External Address"
Changed lines of the file:
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@@
+		)
+	)
+	(text "TODO: External Address\n"
+		(exclude_from_sim no)
+		(at 507.746 26.67 0)
+		(effects
+			(font
+				(size 5.08 5.08)
+			)
 		)
 	)

Commit message: schematic tweaks
Parts:
- removed J2: READOUT, Connector_PinHeader_2.54mm:PinHeader_1x16_P2.54mm_Vertical, symbol Connector:Conn_01x16_Pin
- removed J3: DEVICES, Connector_PinHeader_2.54mm:PinHeader_1x05_P2.54mm_Vertical, symbol Connector:Conn_01x05_Pin
- removed R11, R12: 10k, Resistor_THT:R_Axial_DIN0207_L6.3mm_D2.5mm_P10.16mm_Horizontal, symbol Device:R
- removed SW2: PRG_SELECT, Button_Switch_SMD:SW_DIP_SPSTx08_Slide_9.78x22.5mm_W8.61mm_P2.54mm, symbol Switch:SW_DIP_x08
- removed SW3, SW4: SW_Push, Button_Switch_THT:SW_PUSH_6mm_H5mm, symbol Switch:SW_Push
- added J5: Conn_01x40_Pin, Connector_PinHeader_2.54mm:PinHeader_1x40_P2.54mm_Horizontal, symbol Connector:Conn_01x40_Pin
Connections:
- net +5V: now also J5.1 (Pin_1)
- net A0: now also J5.11 (Pin_11)
- net A1: now also J5.12 (Pin_12)
- net A2: now also J5.13 (Pin_13)
- net A3: now also J5.14 (Pin_14)
- net A4: now also J5.15 (Pin_15)
- net A5: now also J5.16 (Pin_16)
- net A6: now also J5.17 (Pin_17)
- net A7: now also J5.18 (Pin_18)
- net AOUT0: now also J5.2 (Pin_2)
- net AOUT1: now also J5.3 (Pin_3)
- net AOUT2: now also J5.4 (Pin_4)
- net BOUT0: now also J5.6 (Pin_6)
- net BOUT1: now also J5.7 (Pin_7)
- net BOUT2: now also J5.8 (Pin_8)
- net BOUT3: now also J5.9 (Pin_9)
- net CIN: now also J5.10 (Pin_10)
- net Device0: now also J5.36 (Pin_36)
- net Device1: now also J5.37 (Pin_37)
- net Device2: now also J5.38 (Pin_38)
- net Device3: now also J5.39 (Pin_39)
- net GND: now also J5.40 (Pin_40)
- net RESET: now also J5.27 (Pin_27)
- net ROMnCS: now also J5.26 (Pin_26)
- net SignFlag: now also J5.5 (Pin_5)
- net A14: now reaches R10.1, U2.1 (A14)
- net A14: now also J5.25 (Pin_25)
- net A12: now reaches R8.1, U2.2 (A12)
- net A12: now also J5.23 (Pin_23)
- net A10: now reaches R6.1, U2.21 (A10)
- net A10: now also J5.21 (Pin_21)
- net A11: now reaches R7.1, U2.23 (A11)
- net A11: now also J5.22 (Pin_22)
- net A9: now reaches R5.1, U2.24 (A9)
- net A9: now also J5.20 (Pin_20)
- net A8: now reaches R4.1, U2.25 (A8)
- net A8: now also J5.19 (Pin_19)
- net A13: now reaches R9.1, U2.26 (A13)
- net A13: now also J5.24 (Pin_24)
- net MANUALCLK: now reaches SW5.1 (A)
- net MANUALCLK: now also J5.28 (Pin_28)
- new net DATAENTRY: J5.29 (Pin_29)
- no-connect marks 12 -> 11
Other:
- moved on the sheet: J1, R1, R2, R3, SW1

Commit message: PCB
Parts:
- removed U36: ADR_BUFFER, Package_DIP:DIP-14_W7.62mm_Socket, symbol 74xx:74LS125
- added R11, R12, R13, R14: 10K, Resistor_THT:R_Axial_DIN0309_L9.0mm_D3.2mm_P2.54mm_Vertical, symbol Device:R
- R1, R10, R2, R3, R4, R5, R6, R7, R8, R9: footprint Resistor_THT:R_Axial_DIN0207_L6.3mm_D2.5mm_P10.16mm_Horizontal -> Resistor_THT:R_Axial_DIN0309_L9.0mm_D3.2mm_P2.54mm_Vertical
Connections:
- net +5V: now also R11.1, R12.1, R13.1, R14.1
- net A4: now also R14.2
- net A5: now also R13.2
- net A6: now also R12.2
- net A7: now also R11.2
- net ADD: now also U17.1; no longer U18.1
- net ALU0: now also U18.3; no longer U17.3
- net COUT: now also U17.2; no longer U18.2
- net at D20.2 (A): now also U17.3; no longer U18.3
- net at U16.4, U18.10, U18.13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: now also U18.1; no longer U17.1
- net at U12.3: now also U18.2; no longer U17.2
- net DATAENTRY: no longer names the net of J5.29 (Pin_29)
- net MANUALCLK renamed EXTCLK
Other:
- moved on the sheet: U17A, U18A
